File: noise-guy.kicad_sch (KiCad schematic)
At the start: 8 parts, among them J1 Conn_01x03, J2 Conn_01x06, U1 ATtiny10-TS, U2 LM321

Commit message: add pdf for schematics, pcb w/ dimension
Other:
- company: (none) -> Kinoshita Laboratory
- title: (none) -> Noise-guy
Changed lines of the file:
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@@
 (kicad_sch (version 20211123) (generator eeschema)
   (paper "A4")
+  (title_block
+    (title "Noise-guy")
+    (date "2022-11-19")
+    (rev "20221119")
+    (company "Kinoshita Laboratory")
+  )
   (junction (at 161.29 106.68) (diameter 0) (color 0 0 0 0)
   )
